Commit message: Update tool URDF cache and README
Adds URDF files and .obj mesh files for robot tools, including collision and visual meshes.

Also adds a README file explaining the data formats and workflow integration.

File: 250808_cindy_calibration_validation/tool_urdf_cache/BoardTool.urdf (robot description, URDF)
Before this commit: robot BoardTool, 1 links, 0 joints
Links:
- link attached_tool_link: geometry collision mesh filename=9b559ebe-0911-48b2-9e3f-c967b3b849b9.obj; visual mesh filename=d0eb5bbc-6554-45f4-acb9-de08eebcef60.obj

File: 250808_cindy_calibration_validation/tool_urdf_cache/PointTool.urdf (robot description, URDF)
Before this commit: robot PointTool, 1 links, 0 joints
Links:
- link attached_tool_link: geometry collision mesh filename=d47f752e-db0f-476f-bd12-e6c590bd0fb0.obj; visual mesh filename=2e2cc350-2b8b-4f5d-859e-236eb7a7f098.obj
